File: BAgmenzi/power.kicad_sch (KiCad schematic)
At the start: 36 parts, among them J2 DF52-2S-0.8H(21), J3 USB3076-30-A, U10 PESD1USB30, U11 MAX77654BENV+T, U12 TS5A3159AYZPR, U13 TPS7A20xxxDQN, U14 TPS63900

Commit message: added libraries, other changes in sch, started pcb
Parts:
- C47: renamed from C46; footprint (none) -> Capacitor_SMD:C_0402_1005Metric
- C48: renamed from C47; footprint (none) -> Capacitor_SMD:C_0402_1005Metric
- C49: renamed from C48; footprint (none) -> Capacitor_SMD:C_0402_1005Metric
- C50: renamed from C49; footprint (none) -> Capacitor_SMD:C_0402_1005Metric
- C51: renamed from C50; footprint (none) -> Capacitor_SMD:C_0402_1005Metric
- C52: renamed from C51; footprint (none) -> Capacitor_SMD:C_0402_1005Metric
- C53: renamed from C52; footprint (none) -> Capacitor_SMD:C_0402_1005Metric
- C54: renamed from C53; footprint (none) -> Capacitor_SMD:C_0402_1005Metric
- C55: renamed from C54; value C -> 0.1u; footprint (none) -> Capacitor_SMD:C_0402_1005Metric
- C56: renamed from C55; footprint Capacitor_SMD:C_0603_1608Metric -> Capacitor_SMD:C_0402_1005Metric
- C57: renamed from C56; footprint Capacitor_SMD:C_0603_1608Metric -> Capacitor_SMD:C_0402_1005Metric
- C58: renamed from C57; footprint Capacitor_SMD:C_0603_1608Metric -> Capacitor_SMD:C_0402_1005Metric
- C59: renamed from C58; footprint Capacitor_SMD:C_0603_1608Metric -> Capacitor_SMD:C_0402_1005Metric
- C60: renamed from C59; footprint Capacitor_SMD:C_0201_0603Metric -> Capacitor_SMD:C_0402_1005Metric
- L7: footprint C__Users_s-fre_Github_biogap_Hardware_EEG_PcbLib.PcbLib:IND_0805_DFE201210S -> EEG_PcbLib:IND_0805_DFE201210S
- R32, R33, R34, R35, R36, R37, R38, R39, R40, RT1: footprint (none) -> Resistor_SMD:R_0402_1005Metric
- S1: footprint C__Users_s-fre_Github_wulpus_hw_wulpus_acquisition_pcb_PcbLib1.PcbLib:NanoT160BP -> wulpus:NanoT160BP
- U11: footprint C__Users_s-fre_Github_biogap_Hardware_EEG_PcbLib.PcbLib:WLP_30_MAX77654 -> EEG_PcbLib:WLP_30_MAX77654
- U12: footprint BGA6C50P2X3_89X139X50 -> wulpus_pro_acq:BGA6C50P2X3_89X139X50
Connections:
- net PWR.VBAT: no longer C48.1, J2.1, U11.E3 (BAT)
- new net PWR.V_BAT: C48.1, J2.1, U11.E3 (BAT)
Other:
- moved on the sheet: U11C

Commit message: changed VRX rail and deleted U12
Parts:
- removed C55: 0.1u, Capacitor_SMD:C_0402_1005Metric, symbol Device:C
- removed D3: NSR0340HT1G, Diode_SMD:D_SOD-323, symbol Diode:NSR0340HT1G
- removed U12: TS5A3159AYZPR, wulpus_pro_acq:BGA6C50P2X3_89X139X50, symbol TS5A3159AYZPR:TS5A3159AYZPR
- added C32: 0.1u, Capacitor_SMD:C_0402_1005Metric, symbol Device:C
- added D4: NSR20F30NXT5G, NSR20F30NXT5G:DSN2_1, symbol NSR20F30NXT5G:NSR20F30NXT5G
- added JP7: SolderJumper_3_Open, Jumper:SolderJumper-3_P1.3mm_Open_Pad1.0x1.5mm, symbol Jumper:SolderJumper_3_Open
- C56, C57, L8, R37, R38, U14: now not fitted
- C59: value 1u -> 2.2u
- J2: footprint wulpus:DF522S08H21 -> SamacSys:DF522S08H21
- R39: value 0 -> 8.25k; now not fitted
- R40: value 0 -> 1.15k; now not fitted
- U13: value TPS7A20xxxDQN -> TPS7A2033DBVDQN
Connections:
- net GND: now also J3.4, J3.5, C32.2
- net V_LED: now also C32.1
- net V_SYS: now also JP7.3 (B)
- net nRST: now reaches R35.2, U11.A2 (~{RST})
- net at J3.1: now also D4.2 (A)
- net AMUX renamed PMIC_AMUX
- net IRQ renamed PMIC_IRQ
- net PWR.CHGIN renamed CHGIN
- net CHGIN: now also D4.1 (K)
- net PWR.V_BAT renamed V_BAT
- net V_BAT: now also JP7.1 (A)
- net USB_BUS.D_N renamed USB.D_N
- net USB_BUS.D_P renamed USB.D_P
- net V_RX_3.6V: no longer names the net of C57.1, U14.6 (VOUT)
- net V_RX_3.6V: no longer C58.1, U13.4 (IN)
- new net: C58.1, JP7.2 (C), U13.4 (IN)
Other:
- note added: "to generate VRX rail. V_BAT/V_SYS has to be above 3.5V"
- note removed: "to generate V_RX rail: TPS63900 generates 3.6V from V_sys and TPS7A20 LDO cleans it to 3.3V"
- moved on the sheet: C47, C48, C49, C50, C51, C52, C53, C54, C58, C59, C60, FB3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

Commit message: started layout, front v backside
Parts:
- C56, C57, L8, R37, R38, R39, R40, U14: now left out of the parts list
Changed lines of the file:
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@@
 		(unit 1)
 		(exclude_from_sim no)
-		(in_bom yes)
+		(in_bom no)
 		(on_board no)
 		(dnp yes)
@@
 		(unit 1)
 		(exclude_from_sim no)
-		(in_bom yes)
-		(on_board yes)
+		(in_bom no)
+		(on_board no)
 		(dnp yes)
 		(fields_autoplaced yes)
@@
 		(unit 1)
 		(exclude_from_sim no)
-		(in_bom yes)
-		(on_board yes)
+		(in_bom no)
+		(on_board no)
 		(dnp yes)
 		(property "Reference" "L8"
@@
 		(unit 1)
 		(exclude_from_sim no)
-		(in_bom yes)
-		(on_board yes)
+		(in_bom no)
+		(on_board no)
 		(dnp yes)
 		(fields_autoplaced yes)
@@
 		(unit 1)
 		(exclude_from_sim no)
-		(in_bom yes)
-		(on_board yes)
+		(in_bom no)
+		(on_board no)
 		(dnp yes)
 		(property "Reference" "R38"
@@
 		(unit 1)
 		(exclude_from_sim no)
-		(in_bom yes)
-		(on_board yes)
+		(in_bom no)
+		(on_board no)
 		(dnp yes)
 		(fields_autoplaced yes)
@@
 		(unit 1)
 		(exclude_from_sim no)
-		(in_bom yes)
-		(on_board yes)
+		(in_bom no)
+		(on_board no)
 		(dnp yes)
 		(property "Reference" "C56"
@@
 		(unit 1)
 		(exclude_from_sim no)
-		(in_bom yes)
-		(on_board yes)
+		(in_bom no)
+		(on_board no)
 		(dnp yes)
 		(fields_autoplaced yes)

Commit message: started routing, changed enable signals to nRF
Parts:
- added R6: 100k, Resistor_SMD:R_0402_1005Metric, symbol Device:R
Connections:
- net GND: now also R6.2
- net VRX_EN: now also R6.1
- no-connect marks 4 -> 5
Other:
- moved on the sheet: C49
Changed lines of the file:
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@@
 	)
 	(rectangle
-		(start 127 215.9)
-		(end 261.62 275.59)
+		(start 127 218.44)
+		(end 265.43 280.67)
 		(stroke
 			(width 0)
@@
 	)
 	(junction
+		(at 160.02 262.89)
+		(diameter 0)
+		(color 0 0 0 0)
+	)
+	(junction
 		(at 96.52 161.29)
 		(diameter 0)
@@
 	)
 	(no_connect
+		(at 107.95 191.77)
+	)
+	(no_connect
 		(at 351.79 148.59)
 	)
@@
 	(wire
 		(pts
+			(xy 167.64 273.05) (xy 167.64 274.32)
+		)
+		(stroke
+			(width 0)
+			(type default)
+		)
+	)
+	(wire
+		(pts
 			(xy 110.49 330.2) (xy 110.49 328.93)
 		)
@@
 	(wire
 		(pts
+			(xy 167.64 265.43) (xy 167.64 262.89)
+		)
+		(stroke
+			(width 0)
+			(type default)
+		)
+	)
+	(wire
+		(pts
 			(xy 53.34 170.18) (xy 53.34 168.91)
 		)
@@
 	(wire
 		(pts
+			(xy 167.64 262.89) (xy 160.02 262.89)
+		)
+		(stroke
+			(width 0)
+			(type default)
+		)
+	)
+	(wire
+		(pts
 			(xy 152.4 166.37) (xy 148.59 166.37)
 		)
@@
 	(wire
 		(pts
-			(xy 161.29 267.97) (xy 161.29 246.38)
+			(xy 203.2 138.43) (xy 208.28 138.43)
 		)
 		(stroke
@@
 	(wire
 		(pts
-			(xy 203.2 138.43) (xy 208.28 138.43)
+			(xy 107.95 163.83) (xy 101.6 163.83)
 		)
 		(stroke
@@
 	(wire
 		(pts
-			(xy 107.95 163.83) (xy 101.6 163.83)
+			(xy 88.9 346.71) (xy 95.25 346.71)
 		)
 		(stroke
@@
 	(wire
 		(pts
-			(xy 88.9 346.71) (xy 95.25 346.71)
+			(xy 153.67 262.89) (xy 160.02 262.89)
 		)
 		(stroke
@@
 	(wire
 		(pts
+			(xy 160.02 262.89) (xy 160.02 246.38)
+		)
+		(stroke
+			(width 0)
+			(type default)
+		)
+	)
+	(wire
+		(pts
 			(xy 99.06 149.86) (xy 101.6 149.86)
 		)
@@
 	(wire
 		(pts
-			(xy 161.29 246.38) (xy 162.56 246.38)
+			(xy 160.02 246.38) (xy 162.56 246.38)
 		)
 		(stroke
@@
 	(global_label "VRX_EN"
 		(shape input)
-		(at 161.29 267.97 180)
+		(at 153.67 262.89 180)
 		(fields_autoplaced yes)
 		(effects
@@
 		)
 		(property "Intersheetrefs" "${INTERSHEET_REFS}"
-			(at 151.2896 267.97 0)
+			(at 143.6696 262.89 0)
 			(effects
 				(font
@@
 	(symbol
 		(lib_id "power:GND")
+		(at 167.64 274.32 0)
+		(unit 1)
+		(exclude_from_sim no)
+		(in_bom yes)
+		(on_board yes)
+		(dnp no)
+		(fields_autoplaced yes)
+		(property "Reference" "#PWR015"
+			(at 167.64 280.67 0)
+			(effects
+				(font
+					(size 1.27 1.27)
+				)
+				(hide yes)
+			)
+		)
+		(property "Value" "GND"
+			(at 167.64 279.4 0)
+			(effects
+				(font
+					(size 1.27 1.27)
+				)
+			)
+		)
+		(property "Footprint" ""
+			(at 167.64 274.32 0)
+			(effects
+				(font
+					(size 1.27 1.27)
+				)
+				(hide yes)
+			)
+		)
+		(property "Datasheet" ""
+			(at 167.64 274.32 0)
+			(effects
+				(font
+					(size 1.27 1.27)
+				)
+				(hide yes)
+			)
+		)
+		(property "Description" "Power symbol creates a global label with name \"GND\" , ground"
+			(at 167.64 274.32 0)
+			(effects
+				(font
+					(size 1.27 1.27)
+				)
+				(hide yes)
+			)
+		)
+		(pin "1"
+		)
+		(instances
+			(project "BAgmenzi"
+				(path "/8cc4acae-3f14-463c-b0a0-3bc1c8d05954/d463870e-9fcf-4af5-ace7-dfb7bf5f63b9"
+					(reference "#PWR015")
+					(unit 1)
+				)
+			)
+		)
+	)
+	(symbol
+		(lib_id "power:GND")
 		(at 269.24 157.48 0)
 		(unit 1)
@@
 	(symbol
 		(lib_id "Device:R")
+		(at 167.64 269.24 0)
+		(unit 1)
+		(exclude_from_sim no)
+		(in_bom yes)
+		(on_board yes)
+		(dnp no)
+		(property "Reference" "R6"
+			(at 159.512 267.716 0)
+			(effects
+				(font
+					(size 1.27 1.27)
+				)
+				(justify left)
+			)
+		)
+		(property "Value" "100k"
+			(at 159.512 270.256 0)
+			(effects
+				(font
+					(size 1.27 1.27)
+				)
+				(justify left)
+			)
+		)
+		(property "Footprint" "Resistor_SMD:R_0402_1005Metric"
+			(at 165.862 269.24 90)
+			(effects
+				(font
+					(size 1.27 1.27)
+				)
+				(hide yes)
+			)
+		)
+		(property "Datasheet" "~"
+			(at 167.64 269.24 0)
+			(effects
+				(font
+					(size 1.27 1.27)
+				)
+				(hide yes)
+			)
+		)
+		(property "Description" "Resistor"
+			(at 167.64 269.24 0)
+			(effects
+				(font
+					(size 1.27 1.27)
+				)
+				(hide yes)
+			)
+		)
+		(pin "1"
+		)
+		(pin "2"
+		)
+		(instances
+			(project "BAgmenzi"
+				(path "/8cc4acae-3f14-463c-b0a0-3bc1c8d05954/d463870e-9fcf-4af5-ace7-dfb7bf5f63b9"
+					(reference "R6")
+					(unit 1)
+				)
+			)
+		)
+	)
+	(symbol
+		(lib_id "Device:R")
 		(at 41.91 340.36 180)
 		(unit 1)
@@
 	(symbol
 		(lib_id "Device:C")
-		(at 265.43 127 180)
+		(at 265.43 127 0)
+		(mirror x)
 		(unit 1)
 		(exclude_from_sim no)
@@
 		(dnp no)
 		(property "Reference" "C49"
-			(at 261.366 125.73 0)
+			(at 269.494 125.73 0)
 			(effects
 				(font
@@
 		)
 		(property "Value" "1u"
-			(at 261.874 123.444 0)
+			(at 268.986 123.444 0)
 			(effects
 				(font
@@
 		)
 		(property "Footprint" "Capacitor_SMD:C_0402_1005Metric"
-			(at 264.4648 123.19 0)
+			(at 266.3952 123.19 0)
 			(effects
 				(font

Commit message: part numbers added
Parts:
- C32: LCSC Part # (none) -> C161362
- C48, C50: LCSC Part # (none) -> C23733
- C49, C51, C58: LCSC Part # (none) -> C20441333
- C53: LCSC Part # (none) -> C2190182
- C56: LCSC Part # (none) -> C15525
- C59: LCSC Part # (none) -> C12530
- C60: LCSC Part # (none) -> C1713
- D4: LCSC Part # (none) -> C145508
- J2: LCSC Part # (none) -> C82431
- J3: LCSC Part # (none) -> C6007475
- R32, R33: LCSC Part # (none) -> C423829
- R34, R35, R6: LCSC Part # (none) -> C723496
- R36: value 10K -> 10k; LCSC Part # (none) -> C270305
- S1: LCSC Part # (none) -> C2760983
- U11: LCSC Part # (none) -> C3189129
Changed lines of the file:
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@@
 			)
 		)
+		(property "LCSC Part #" "C2190182"
+			(at 213.36 146.05 90)
+			(effects
+				(font
+					(size 1.27 1.27)
+				)
+				(hide yes)
+			)
+		)
 		(pin "2"
 		)
@@
 			)
 		)
+		(property "LCSC Part #" "C3189129"
+			(at 331.47 146.05 0)
+			(effects
+				(font
+					(size 1.27 1.27)
+				)
+				(hide yes)
+			)
+		)
 		(pin "E1"
 		)
@@
 			)
 		)
+		(property "LCSC Part #" "C723496"
+			(at 68.58 154.94 0)
+			(effects
+				(font
+					(size 1.27 1.27)
+				)
+				(hide yes)
+			)
+		)
 		(pin "2"
 		)
@@
 			)
 		)
+		(property "LCSC Part #" "C3189129"
+			(at 243.84 135.89 0)
+			(effects
+				(font
+					(size 1.27 1.27)
+				)
+				(hide yes)
+			)
+		)
 		(pin "E1"
 		)
@@
 			)
 		)
+		(property "LCSC Part #" "C23733"
+			(at 97.79 127 0)
+			(effects
+				(font
+					(size 1.27 1.27)
+				)
+				(hide yes)
+			)
+		)
 		(pin "2"
 		)
@@
 			)
 		)
+		(property "LCSC Part #" "C145508"
+			(at 105.41 43.18 0)
+			(effects
+				(font
+					(size 1.27 1.27)
+				)
+				(hide yes)
+			)
+		)
 		(pin "1"
 		)
@@
 			)
 		)
+		(property "LCSC Part #" "C12530"
+			(at 182.88 248.92 0)
+			(effects
+				(font
+					(size 1.27 1.27)
+				)
+				(hide yes)
+			)
+		)
 		(pin "2"
 		)
@@
 			)
 		)
+		(property "LCSC Part #" "C1713"
+			(at 219.71 252.73 0)
+			(effects
+				(font
+					(size 1.27 1.27)
+				)
+				(hide yes)
+			)
+		)
 		(pin "2"
 		)
@@
 			)
 		)
+		(property "LCSC Part #" "C723496"
+			(at 167.64 269.24 0)
+			(effects
+				(font
+					(size 1.27 1.27)
+				)
+				(hide yes)
+			)
+		)
 		(pin "1"
 		)
@@
 			)
 		)
+		(property "LCSC Part #" "C3189129"
+			(at 128.27 130.81 0)
+			(effects
+				(font
+					(size 1.27 1.27)
+				)
+				(hide yes)
+			)
+		)
 		(pin "E1"
 		)
@@
 			)
 		)
+		(property "LCSC Part #" "C15525"
+			(at 54.61 323.85 0)
+			(effects
+				(font
+					(size 1.27 1.27)
+				)
+				(hide yes)
+			)
+		)
 		(pin "2"
 		)
@@
 			)
 		)
+		(property "LCSC Part #" "C6007475"
+			(at 142.24 52.07 0)
+			(effects
+				(font
+					(size 1.27 1.27)
+				)
+				(hide yes)
+			)
+		)
 		(pin "1"
 		)
@@
 			)
 		)
+		(property "LCSC Part #" "C20441333"
+			(at 265.43 127 0)
+			(effects
+				(font
+					(size 1.27 1.27)
+				)
+				(hide yes)
+			)
+		)
 		(pin "2"
 		)
@@
 			)
 		)
+		(property "LCSC Part #" "C423829"
+			(at 96.52 153.67 0)
+			(effects
+				(font
+					(size 1.27 1.27)
+				)
+				(hide yes)
+			)
+		)
 		(pin "2"
 		)
@@
 			)
 		)
+		(property "LCSC Part #" "C2760983"
+			(at 69.85 184.15 0)
+			(effects
+				(font
+					(size 1.27 1.27)
+				)
+				(hide yes)
+			)
+		)
 		(pin "1"
 		)
@@
 			)
 		)
+		(property "LCSC Part #" "C82431"
+			(at 198.12 36.83 0)
+			(effects
+				(font
+					(size 1.27 1.27)
+				)
+				(hide yes)
+			)
+		)
 		(pin "3"
 		)
@@
 			)
 		)
+		(property "LCSC Part #" "C20441333"
+			(at 151.13 247.65 0)
+			(effects
+				(font
+					(size 1.27 1.27)
+				)
+				(hide yes)
+			)
+		)
 		(pin "2"
 		)
@@
 			)
 		)
+		(property "LCSC Part #" "C723496"
+			(at 58.42 154.94 0)
+			(effects
+				(font
+					(size 1.27 1.27)
+				)
+				(hide yes)
+			)
+		)
 		(pin "2"
 		)
@@
 			)
 		)
-		(property "Value" "10K"
+		(property "Value" "10k"
 			(at 156.21 162.56 90)
 			(effects
@@
 			)
 		)
+		(property "LCSC Part #" "C270305"
+			(at 156.21 166.37 90)
+			(effects
+				(font
+					(size 1.27 1.27)
+				)
+				(hide yes)
+			)
+		)
 		(pin "2"
 		)
@@
 			)
 		)
+		(property "LCSC Part #" "C20441333"
+			(at 158.75 129.54 0)
+			(effects
+				(font
+					(size 1.27 1.27)
+				)
+				(hide yes)
+			)
+		)
 		(pin "2"
 		)
@@
 			)
 		)
+		(property "LCSC Part #" "C23733"
+			(at 86.36 128.27 0)
+			(effects
+				(font
+					(size 1.27 1.27)
+				)
+				(hide yes)
+			)
+		)
 		(pin "2"
 		)
@@
 			)
 		)
+		(property "LCSC Part #" "C161362"
+			(at 279.4 152.4 0)
+			(effects
+				(font
+					(size 1.27 1.27)
+				)
+				(hide yes)
+			)
+		)
 		(pin "2"
 		)
@@
 			(at 101.6 153.67 0)
 			(effects
+				(font
+					(size 1.27 1.27)
+				)
+				(hide yes)
+			)
+		)
+		(property "LCSC Part #" "C423829"
+			(at 101.6 153.67 0)
+			(effects
