File: BAgmenzi/rx.kicad_sch (KiCad schematic)
At the start: 30 parts, among them IC1 TPL0501-100RSER, U2 AD8338ACPZ-R7, U3 OPA836IDBVT, U4 OPA836IDBVT

Commit message: added polyCMUT footprint, changed enables, more compact
Parts:
- removed TP2: vga_vref, TestPoint:TestPoint_Pad_D2.0mm, symbol Connector:TestPoint
- removed TP6: TestPoint, TestPoint:TestPoint_Pad_D2.0mm, symbol Connector:TestPoint
- added C67: 47u, Capacitor_SMD:C_0402_1005Metric, symbol Device:C
- C25: value 10nF -> 1.5n
- C34: value 1n -> 3.3n
- R10: value 100 -> 0
- R11: value 400 -> 1
- R7: value 2k -> 200
- R8: value 2k -> 1k
Connections:
- net GND: now also C67.1
- net V_RX: now also C67.2
Changed lines of the file:
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@@
 	)
 	(junction
-		(at 222.25 151.13)
-		(diameter 0)
-		(color 0 0 0 0)
-	)
-	(junction
 		(at 234.95 82.55)
 		(diameter 0)
@@
 	)
 	(junction
+		(at 36.83 43.18)
+		(diameter 0)
+		(color 0 0 0 0)
+	)
+	(junction
 		(at 317.5 69.85)
 		(diameter 0)
@@
 	)
 	(junction
-		(at 360.68 69.85)
+		(at 36.83 34.29)
 		(diameter 0)
 		(color 0 0 0 0)
 	)
 	(junction
-		(at 179.07 80.01)
+		(at 360.68 69.85)
 		(diameter 0)
 		(color 0 0 0 0)
@@
 	(wire
 		(pts
-			(xy 179.07 80.01) (xy 180.34 80.01)
+			(xy 177.8 80.01) (xy 180.34 80.01)
 		)
 		(stroke
@@
 	(wire
 		(pts
+			(xy 36.83 34.29) (xy 48.26 34.29)
+		)
+		(stroke
+			(width 0)
+			(type default)
+		)
+	)
+	(wire
+		(pts
 			(xy 76.2 85.09) (xy 80.01 85.09)
 		)
@@
 	(wire
 		(pts
-			(xy 222.25 151.13) (xy 227.33 151.13)
-		)
-		(stroke
-			(width 0)
-			(type default)
-		)
-	)
-	(wire
-		(pts
 			(xy 180.34 39.37) (xy 186.69 39.37)
 		)
@@
 	(wire
 		(pts
-			(xy 177.8 80.01) (xy 179.07 80.01)
-		)
-		(stroke
-			(width 0)
-			(type default)
-		)
-	)
-	(wire
-		(pts
 			(xy 81.28 50.8) (xy 81.28 67.31)
 		)
@@
 	(wire
 		(pts
-			(xy 220.98 151.13) (xy 222.25 151.13)
+			(xy 220.98 151.13) (xy 227.33 151.13)
 		)
 		(stroke
@@
 	(wire
 		(pts
+			(xy 36.83 43.18) (xy 48.26 43.18)
+		)
+		(stroke
+			(width 0)
+			(type default)
+		)
+	)
+	(wire
+		(pts
 			(xy 278.13 46.99) (xy 332.74 46.99)
 		)
@@
 	(wire
 		(pts
+			(xy 48.26 41.91) (xy 48.26 43.18)
+		)
+		(stroke
+			(width 0)
+			(type default)
+		)
+	)
+	(wire
+		(pts
 			(xy 120.65 69.85) (xy 120.65 50.8)
 		)
@@
 			)
 		)
-		(property "Value" "2k"
+		(property "Value" "1k"
 			(at 99.06 48.514 90)
 			(effects
@@
 			)
 		)
-		(property "Value" "1n"
+		(property "Value" "3.3n"
 			(at 254 161.2899 0)
 			(effects
@@
 			)
 		)
-		(property "Value" "2k"
+		(property "Value" "200"
 			(at 74.93 38.1 90)
 			(effects
@@
 			)
 		)
-		(property "Value" "10nF"
+		(property "Value" "1.5n"
 			(at 67.31 36.83 90)
 			(effects
@@
 			)
 		)
-		(property "Value" "100"
+		(property "Value" "0"
 			(at 71.12 68.58 90)
 			(effects
@@
 	)
 	(symbol
-		(lib_id "Connector:TestPoint")
-		(at 179.07 80.01 180)
-		(unit 1)
-		(exclude_from_sim no)
-		(in_bom yes)
-		(on_board yes)
-		(dnp no)
-		(property "Reference" "TP2"
-			(at 184.658 87.884 0)
-			(effects
-				(font
-					(size 1.27 1.27)
-				)
-				(justify left)
-			)
-		)
-		(property "Value" "vga_vref"
-			(at 188.468 85.852 0)
-			(effects
-				(font
-					(size 1.27 1.27)
-				)
-				(justify left)
-			)
-		)
-		(property "Footprint" "TestPoint:TestPoint_Pad_D2.0mm"
-			(at 173.99 80.01 0)
-			(effects
-				(font
-					(size 1.27 1.27)
-				)
-				(hide yes)
-			)
-		)
-		(property "Datasheet" "~"
-			(at 173.99 80.01 0)
-			(effects
-				(font
-					(size 1.27 1.27)
-				)
-				(hide yes)
-			)
-		)
-		(property "Description" "test point"
-			(at 179.07 80.01 0)
-			(effects
-				(font
-					(size 1.27 1.27)
-				)
-				(hide yes)
-			)
-		)
-		(pin "1"
-		)
-		(instances
-			(project "BAgmenzi"
-				(path "/8cc4acae-3f14-463c-b0a0-3bc1c8d05954/a3b6f7aa-6ef7-488e-b797-42706d211223"
-					(reference "TP2")
-					(unit 1)
-				)
-			)
-		)
-	)
-	(symbol
 		(lib_id "Device:C")
 		(at 80.01 90.17 180)
@@
 			)
 		)
-		(property "Value" "400"
+		(property "Value" "1"
 			(at 251.46 73.6599 0)
 			(effects
@@
 	(symbol
 		(lib_id "Device:C")
-		(at 184.15 69.85 90)
+		(at 48.26 38.1 180)
 		(unit 1)
 		(exclude_from_sim no)
@@
 		(on_board yes)
 		(dnp no)
-		(fields_autoplaced yes)
-		(property "Reference" "C27"
-			(at 184.15 62.23 90)
+		(property "Reference" "C67"
+			(at 51.308 36.83 0)
 			(effects
 				(font
 					(size 1.27 1.27)
 				)
+				(justify right)
 			)
 		)
-		(property "Value" "1n"
-			(at 184.15 64.77 90)
+		(property "Value" "47u"
+			(at 51.308 39.37 0)
 			(effects
 				(font
 					(size 1.27 1.27)
 				)
+				(justify right)
 			)
 		)
 		(property "Footprint" "Capacitor_SMD:C_0402_1005Metric"
-			(at 187.96 68.8848 0)
+			(at 47.2948 34.29 0)
 			(effects
 				(font
@@
 		)
 		(property "Datasheet" "~"
-			(at 184.15 69.85 0)
+			(at 48.26 38.1 0)
 			(effects
 				(font
@@
 		)
 		(property "Description" "Unpolarized capacitor"
-			(at 184.15 69.85 0)
+			(at 48.26 38.1 0)
 			(effects
 				(font
@@
 		)
 		(instances
-			(project ""
+			(project "BAgmenzi"
 				(path "/8cc4acae-3f14-463c-b0a0-3bc1c8d05954/a3b6f7aa-6ef7-488e-b797-42706d211223"
-					(reference "C27")
+					(reference "C67")
 					(unit 1)
 				)
@@
 	(symbol
 		(lib_id "Device:C")
-		(at 184.15 80.01 90)
+		(at 184.15 69.85 90)
 		(unit 1)
 		(exclude_from_sim no)
@@
 		(on_board yes)
 		(dnp no)
-		(property "Reference" "C30"
-			(at 184.15 74.168 90)
+		(fields_autoplaced yes)
+		(property "Reference" "C27"
+			(at 184.15 62.23 90)
 			(effects
 				(font
@@
 		)
 		(property "Value" "1n"
-			(at 183.896 76.454 90)
+			(at 184.15 64.77 90)
 			(effects
 				(font
@@
 		)
 		(property "Footprint" "Capacitor_SMD:C_0402_1005Metric"
-			(at 187.96 79.0448 0)
+			(at 187.96 68.8848 0)
 			(effects
 				(font
@@
 		)
 		(property "Datasheet" "~"
-			(at 184.15 80.01 0)
+			(at 184.15 69.85 0)
 			(effects
 				(font
@@
 		)
 		(property "Description" "Unpolarized capacitor"
-			(at 184.15 80.01 0)
+			(at 184.15 69.85 0)
 			(effects
 				(font
@@
 		)
 		(instances
-			(project "BAgmenzi"
+			(project ""
 				(path "/8cc4acae-3f14-463c-b0a0-3bc1c8d05954/a3b6f7aa-6ef7-488e-b797-42706d211223"
-					(reference "C30")
+					(reference "C27")
 					(unit 1)
 				)
@@
 	)
 	(symbol
-		(lib_id "Connector:TestPoint")
-		(at 222.25 151.13 0)
+		(lib_id "Device:C")
+		(at 184.15 80.01 90)
 		(unit 1)
 		(exclude_from_sim no)
@@
 		(on_board yes)
 		(dnp no)
-		(property "Reference" "TP6"
-			(at 218.186 143.764 0)
+		(property "Reference" "C30"
+			(at 184.15 74.168 90)
 			(effects
 				(font
 					(size 1.27 1.27)
 				)
-				(justify left)
 			)
 		)
-		(property "Value" "TestPoint"
-			(at 218.186 145.542 0)
+		(property "Value" "1n"
+			(at 183.896 76.454 90)
 			(effects
 				(font
 					(size 1.27 1.27)
 				)
-				(justify left)
 			)
 		)
-		(property "Footprint" "TestPoint:TestPoint_Pad_D2.0mm"
-			(at 227.33 151.13 0)
+		(property "Footprint" "Capacitor_SMD:C_0402_1005Metric"
+			(at 187.96 79.0448 0)
 			(effects
 				(font
@@
 		)
 		(property "Datasheet" "~"
-			(at 227.33 151.13 0)
+			(at 184.15 80.01 0)
 			(effects
 				(font
@@
 			)
 		)
-		(property "Description" "test point"
-			(at 222.25 151.13 0)
+		(property "Description" "Unpolarized capacitor"
+			(at 184.15 80.01 0)
 			(effects
 				(font
@@
 		(pin "1"
 		)
+		(pin "2"
+		)
 		(instances
-			(project ""
+			(project "BAgmenzi"
 				(path "/8cc4acae-3f14-463c-b0a0-3bc1c8d05954/a3b6f7aa-6ef7-488e-b797-42706d211223"
-					(reference "TP6")
+					(reference "C30")
 					(unit 1)
 				)

Commit message: part numbers added
Parts:
- C19, C21, C23, C31: LCSC Part # (none) -> C12530
- C20, C22, C24: LCSC Part # (none) -> C161362
- C25: LCSC Part # (none) -> C23967
- C26: LCSC Part # (none) -> C783011
- C27, C30: LCSC Part # (none) -> C3832658
- C28: LCSC Part # (none) -> C2927434
- C29: LCSC Part # (none) -> C2168619
- C34: LCSC Part # (none) -> C2190182
- C67: footprint Capacitor_SMD:C_0402_1005Metric -> Capacitor_SMD:C_0603_1608Metric
- IC1: LCSC Part # (none) -> C1539758
- R10: LCSC Part # (none) -> C364372
- R11: LCSC Part # (none) -> C22369188
- R12: LCSC Part # (none) -> C880417
- R13: LCSC Part # (none) -> C270305
- R15: LCSC Part # (none) -> C22356209
- R16: LCSC Part # (none) -> C560348
- R7: LCSC Part # (none) -> C560339
- R8: LCSC Part # (none) -> C606165
- R9: LCSC Part # (none) -> C22469448
- U2: LCSC Part # (none) -> C578701
- U3, U4: LCSC Part # (none) -> C2057515
