File: BAgmenzi/rx.kicad_sch (KiCad schematic)
At the start: 29 parts, among them IC1 TPL0501-100RSER, U2 AD8338ACPZ-R7, U3 OPA836IDBVT, U4 OPA836IDBVT

Commit message: LCSC parts complete, changed L5andL6 footprint
Parts:
- C19, C21, C23, C31: LCSC Part # C12530 -> C77002
- C20, C22, C24: LCSC Part # C161362 -> C169842
- C26: LCSC Part # C783011 -> C76900
- C27, C30: LCSC Part # C3832658 -> C76947
- C28: LCSC Part # C2927434 -> C2167243
- C29: LCSC Part # C2168619 -> C597012
- C34: LCSC Part # C2190182 -> C26404
- C67: LCSC Part # (none) -> C730416
- R10: LCSC Part # C364372 -> C190119
- R11: LCSC Part # C22369188 -> C2077765
- R12: LCSC Part # C880417 -> C482184
- R13: LCSC Part # C270305 -> C191984
- R15: LCSC Part # C22356209 -> C25866
- R16: LCSC Part # C560348 -> C2074348
- R7: LCSC Part # C560339 -> C25087
- R8: LCSC Part # C606165 -> C11702
- R9: value 400 -> 402; LCSC Part # C22469448 -> C41042
Changed lines of the file:
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@@
 			)
 		)
-		(property "LCSC Part #" "C161362"
+		(property "LCSC Part #" "C169842 "
 			(at 36.83 39.37 0)
 			(effects
@@
 			)
 		)
-		(property "LCSC Part #" "C161362"
+		(property "LCSC Part #" "C169842 "
 			(at 186.69 35.56 0)
 			(effects
@@
 			)
 		)
-		(property "LCSC Part #" "C606165"
+		(property "LCSC Part #" "C11702 "
 			(at 99.06 50.8 90)
 			(effects
@@
 			)
 		)
-		(property "LCSC Part #" "C12530"
+		(property "LCSC Part #" "C77002 "
 			(at 307.34 36.83 0)
 			(effects
@@
 			)
 		)
-		(property "LCSC Part #" "C783011"
+		(property "LCSC Part #" "C76900 "
 			(at 99.06 41.91 90)
 			(effects
@@
 			)
 		)
-		(property "LCSC Part #" "C2190182"
+		(property "LCSC Part #" "C26404 "
 			(at 250.19 160.02 0)
 			(effects
@@
 			)
 		)
-		(property "LCSC Part #" "C22356209"
+		(property "LCSC Part #" "C25866 "
 			(at 231.14 151.13 90)
 			(effects
@@
 			)
 		)
-		(property "LCSC Part #" "C560339"
+		(property "LCSC Part #" "C25087 "
 			(at 74.93 41.91 90)
 			(effects
@@
 			)
 		)
-		(property "Value" "400"
+		(property "Value" "402"
 			(at 350.52 66.04 90)
 			(effects
@@
 			)
 		)
-		(property "LCSC Part #" "C22469448"
+		(property "LCSC Part #" "C41042 "
 			(at 350.52 69.85 90)
 			(effects
@@
 			)
 		)
-		(property "LCSC Part #" "C364372"
+		(property "LCSC Part #" "C190119 "
 			(at 71.12 72.39 90)
 			(effects
@@
 			)
 		)
-		(property "LCSC Part #" "C560348"
+		(property "LCSC Part #" "C2074348 "
 			(at 191.77 175.26 90)
 			(effects
@@
 			)
 		)
-		(property "LCSC Part #" "C161362"
+		(property "LCSC Part #" "C169842 "
 			(at 318.77 36.83 0)
 			(effects
@@
 			)
 		)
-		(property "LCSC Part #" "C2168619"
+		(property "LCSC Part #" "C597012 "
 			(at 360.68 76.2 0)
 			(effects
@@
 			)
 		)
-		(property "LCSC Part #" "C12530"
+		(property "LCSC Part #" "C77002 "
 			(at 80.01 90.17 0)
 			(effects
@@
 			)
 		)
-		(property "LCSC Part #" "C880417"
+		(property "LCSC Part #" "C482184 "
 			(at 80.01 80.01 0)
 			(effects
@@
 			)
 		)
-		(property "LCSC Part #" "C12530"
+		(property "LCSC Part #" "C77002 "
 			(at 175.26 35.56 0)
 			(effects
@@
 			)
 		)
-		(property "LCSC Part #" "C22369188"
+		(property "LCSC Part #" "C2077765 "
 			(at 248.92 72.39 0)
 			(effects
@@
 			)
 		)
-		(property "LCSC Part #" "C270305"
+		(property "LCSC Part #" "C191984 "
 			(at 307.34 95.25 90)
 			(effects
@@
 			)
 		)
-		(property "LCSC Part #" "C2927434"
+		(property "LCSC Part #" "C2167243 "
 			(at 58.42 72.39 90)
 			(effects
@@
 			)
 		)
+		(property "LCSC Part #" "C730416"
+			(at 48.26 38.1 0)
+			(effects
+				(font
+					(size 1.27 1.27)
+				)
+				(hide yes)
+			)
+		)
 		(pin "1"
 		)
@@
 			)
 		)
-		(property "LCSC Part #" "C3832658"
+		(property "LCSC Part #" "C76947 "
 			(at 184.15 69.85 90)
 			(effects
@@
 			)
 		)
-		(property "LCSC Part #" "C3832658"
+		(property "LCSC Part #" "C76947 "
 			(at 184.15 80.01 90)
 			(effects
@@
 			)
 		)
-		(property "LCSC Part #" "C12530"
+		(property "LCSC Part #" "C77002 "
 			(at 25.4 39.37 0)
 			(effects

Commit message: corrected LCSC numbers, other changes, Testpoints
Parts:
- removed TP3: filt_shdn_en, symbol Connector:TestPoint
- C19, C21, C23, C31: LCSC Part # C77002 -> C77002
- C20, C22, C24: LCSC Part # C169842 -> C1525
- C26: LCSC Part # C76900 -> C76900
- C27, C30: LCSC Part # C76947 -> C76947
- C28: LCSC Part # C2167243 -> C2167243
- C29: LCSC Part # C597012 -> C1546
- C34: LCSC Part # C26404 -> C26404
- R10: LCSC Part # C190119 -> C190119
- R11: LCSC Part # C2077765 -> C2077765
- R12: LCSC Part # C482184 -> C482184
- R13: LCSC Part # C191984 -> C191984
- R15: LCSC Part # C25866 -> C25866
- R16: LCSC Part # C2074348 -> C2074348
- R7: LCSC Part # C25087 -> C25087
- R8: LCSC Part # C11702 -> C11702
- R9: LCSC Part # C41042 -> C41042
Changed lines of the file:
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@@
 			)
 		)
-		(property "LCSC Part #" "C169842 "
+		(property "LCSC Part #" "C1525"
 			(at 36.83 39.37 0)
 			(effects
@@
 			)
 		)
-		(property "LCSC Part #" "C169842 "
+		(property "LCSC Part #" "C1525"
 			(at 186.69 35.56 0)
 			(effects
@@
 			)
 		)
-		(property "LCSC Part #" "C11702 "
+		(property "LCSC Part #" "C11702"
 			(at 99.06 50.8 90)
 			(effects
@@
 			)
 		)
-		(property "LCSC Part #" "C77002 "
+		(property "LCSC Part #" "C77002"
 			(at 307.34 36.83 0)
 			(effects
@@
 			)
 		)
-		(property "LCSC Part #" "C76900 "
+		(property "LCSC Part #" "C76900"
 			(at 99.06 41.91 90)
 			(effects
@@
 			)
 		)
-		(property "LCSC Part #" "C26404 "
+		(property "LCSC Part #" "C26404"
 			(at 250.19 160.02 0)
 			(effects
@@
 			)
 		)
-		(property "LCSC Part #" "C25866 "
+		(property "LCSC Part #" "C25866"
 			(at 231.14 151.13 90)
 			(effects
@@
 			)
 		)
-		(property "LCSC Part #" "C25087 "
+		(property "LCSC Part #" "C25087"
 			(at 74.93 41.91 90)
 			(effects
@@
 			)
 		)
-		(property "LCSC Part #" "C41042 "
+		(property "LCSC Part #" "C41042"
 			(at 350.52 69.85 90)
 			(effects
@@
 			)
 		)
-		(property "LCSC Part #" "C190119 "
+		(property "LCSC Part #" "C190119"
 			(at 71.12 72.39 90)
 			(effects
@@
 			)
 		)
-		(property "LCSC Part #" "C2074348 "
+		(property "LCSC Part #" "C2074348"
 			(at 191.77 175.26 90)
 			(effects
@@
 			)
 		)
-		(property "LCSC Part #" "C169842 "
+		(property "LCSC Part #" "C1525"
 			(at 318.77 36.83 0)
 			(effects
@@
 	)
 	(symbol
-		(lib_id "Connector:TestPoint")
-		(at 299.72 95.25 180)
-		(unit 1)
-		(exclude_from_sim no)
-		(in_bom yes)
-		(on_board yes)
-		(dnp no)
-		(property "Reference" "TP3"
-			(at 305.308 103.124 0)
-			(effects
-				(font
-					(size 1.27 1.27)
-				)
-				(justify left)
-			)
-		)
-		(property "Value" "filt_shdn_en"
-			(at 309.118 101.092 0)
-			(effects
-				(font
-					(size 1.27 1.27)
-				)
-				(justify left)
-			)
-		)
-		(property "Footprint" ""
-			(at 294.64 95.25 0)
-			(effects
-				(font
-					(size 1.27 1.27)
-				)
-				(hide yes)
-			)
-		)
-		(property "Datasheet" "~"
-			(at 294.64 95.25 0)
-			(effects
-				(font
-					(size 1.27 1.27)
-				)
-				(hide yes)
-			)
-		)
-		(property "Description" "test point"
-			(at 299.72 95.25 0)
-			(effects
-				(font
-					(size 1.27 1.27)
-				)
-				(hide yes)
-			)
-		)
-		(pin "1"
-		)
-		(instances
-			(project "BAgmenzi"
-				(path "/8cc4acae-3f14-463c-b0a0-3bc1c8d05954/a3b6f7aa-6ef7-488e-b797-42706d211223"
-					(reference "TP3")
-					(unit 1)
-				)
-			)
-		)
-	)
-	(symbol
 		(lib_id "Device:C")
 		(at 360.68 76.2 180)
@@
 			)
 		)
-		(property "LCSC Part #" "C597012 "
+		(property "LCSC Part #" "C1546"
 			(at 360.68 76.2 0)
 			(effects
@@
 			)
 		)
-		(property "LCSC Part #" "C77002 "
+		(property "LCSC Part #" "C77002"
 			(at 80.01 90.17 0)
 			(effects
@@
 			)
 		)
-		(property "LCSC Part #" "C482184 "
+		(property "LCSC Part #" "C482184"
 			(at 80.01 80.01 0)
 			(effects
@@
 			)
 		)
-		(property "LCSC Part #" "C77002 "
+		(property "LCSC Part #" "C77002"
 			(at 175.26 35.56 0)
 			(effects
@@
 			)
 		)
-		(property "LCSC Part #" "C2077765 "
+		(property "LCSC Part #" "C2077765"
 			(at 248.92 72.39 0)
 			(effects
@@
 			)
 		)
-		(property "LCSC Part #" "C191984 "
+		(property "LCSC Part #" "C191984"
 			(at 307.34 95.25 90)
 			(effects
@@
 			)
 		)
-		(property "LCSC Part #" "C2167243 "
+		(property "LCSC Part #" "C2167243"
 			(at 58.42 72.39 90)
 			(effects
@@
 			)
 		)
-		(property "LCSC Part #" "C76947 "
+		(property "LCSC Part #" "C76947"
 			(at 184.15 69.85 90)
 			(effects
@@
 			)
 		)
-		(property "LCSC Part #" "C76947 "
+		(property "LCSC Part #" "C76947"
 			(at 184.15 80.01 90)
 			(effects
@@
 			)
 		)
-		(property "LCSC Part #" "C77002 "
+		(property "LCSC Part #" "C77002"
 			(at 25.4 39.37 0)
 			(effects
