File: BAgmenzi/msp.kicad_sch (KiCad schematic)
At the start: 30 parts, among them J1 Conn_01x07, U1 MSP430FR5043IRGCT, X1 FY0800018, X2 ABS07-32.768KHZ-9-T, Y1 AWSCR-8.00CV-T

Commit message: LCSC parts complete, changed L5andL6 footprint
Parts:
- C1, C2, C5, C6: LCSC Part # C3832658 -> C76947
- C10, C11, C12: LCSC Part # C161362 -> C169842
- C13, C14, C15, C16, C17, C18: LCSC Part # C2176190 -> C161305
- C3, C4: LCSC Part # (none) -> C730416
- C7, C8, C9: LCSC Part # C12530 -> C77002
- L1, L2: LCSC Part # C2661857 -> C41556732
- R1: LCSC Part # C880417 -> C482184
- R2, R3: LCSC Part # C473625 -> C413126
- R4, R5: LCSC Part # C161362 -> C114765
- U1: LCSC Part # C3189129 -> C5218420
- X1: LCSC Part # C6951614 -> C6951614
- X2: LCSC Part # C179635 -> C179635
- Y1: LCSC Part # C2650764 -> C2650764
Changed lines of the file:
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@@
 			)
 		)
-		(property "LCSC Part #" "C2661857"
+		(property "LCSC Part #" "C41556732 "
 			(at 316.23 201.93 0)
 			(effects
@@
 			)
 		)
-		(property "LCSC Part #" "C161362"
+		(property "LCSC Part #" "C169842 "
 			(at 345.44 240.03 90)
 			(effects
@@
 			)
 		)
+		(property "LCSC Part #" "C730416"
+			(at 307.34 191.77 0)
+			(effects
+				(font
+					(size 1.27 1.27)
+				)
+				(hide yes)
+			)
+		)
 		(pin "2"
 		)
@@
 			)
 		)
-		(property "LCSC Part #" "C3189129"
+		(property "LCSC Part #" "C5218420 "
 			(at 163.83 91.44 0)
 			(effects
@@
 			)
 		)
-		(property "LCSC Part #" "C161362"
+		(property "LCSC Part #" "C114765 "
 			(at 138.43 232.41 90)
 			(effects
@@
 			)
 		)
-		(property "LCSC Part #" "C2176190"
+		(property "LCSC Part #" "C161305 "
 			(at 41.91 264.16 90)
 			(effects
@@
 			)
 		)
-		(property "LCSC Part #" "C12530"
+		(property "LCSC Part #" "C77002 "
 			(at 312.42 231.14 90)
 			(effects
@@
 			)
 		)
-		(property "LCSC Part #" "C161362"
+		(property "LCSC Part #" "C169842 "
 			(at 381 241.3 90)
 			(effects
@@
 			)
 		)
-		(property "LCSC Part #" "C161362"
+		(property "LCSC Part #" "C169842 "
 			(at 312.42 240.03 90)
 			(effects
@@
 			)
 		)
-		(property "LCSC Part #" "C880417"
+		(property "LCSC Part #" "C482184 "
 			(at 369.57 41.91 0)
 			(effects
@@
 			)
 		)
-		(property "LCSC Part #" " C473625"
+		(property "LCSC Part #" "C413126 "
 			(at 265.43 67.31 0)
 			(effects
@@
 			)
 		)
-		(property "LCSC Part #" "C3832658"
+		(property "LCSC Part #" "C76947 "
 			(at 323.85 184.15 0)
 			(effects
@@
 			)
 		)
-		(property "LCSC Part #" "C6951614"
+		(property "LCSC Part #" "C6951614 "
 			(at 31.75 213.36 0)
 			(effects
@@
 			)
 		)
-		(property "LCSC Part #" "C2176190"
+		(property "LCSC Part #" "C161305 "
 			(at 38.1 229.87 90)
 			(effects
@@
 			)
 		)
-		(property "LCSC Part #" "C2176190"
+		(property "LCSC Part #" "C161305 "
 			(at 123.19 257.81 90)
 			(effects
@@
 			)
 		)
-		(property "LCSC Part #" "C2650764"
+		(property "LCSC Part #" "C2650764 "
 			(at 114.3 240.03 0)
 			(effects
@@
 			)
 		)
-		(property "LCSC Part #" " C473625"
+		(property "LCSC Part #" "C413126 "
 			(at 279.4 67.31 0)
 			(effects
@@
 			)
 		)
-		(property "LCSC Part #" "C3832658"
+		(property "LCSC Part #" "C76947 "
 			(at 307.34 184.15 0)
 			(effects
@@
 			)
 		)
-		(property "LCSC Part #" "C2176190"
+		(property "LCSC Part #" "C161305 "
 			(at 38.1 199.39 90)
 			(effects
@@
 			)
 		)
-		(property "LCSC Part #" "C179635"
+		(property "LCSC Part #" "C179635 "
 			(at 48.26 261.62 90)
 			(effects
@@
 			)
 		)
-		(property "LCSC Part #" "C161362"
+		(property "LCSC Part #" "C114765 "
 			(at 55.88 199.39 90)
 			(effects
@@
 			)
 		)
+		(property "LCSC Part #" "C730416"
+			(at 323.85 191.77 0)
+			(effects
+				(font
+					(size 1.27 1.27)
+				)
+				(hide yes)
+			)
+		)
 		(pin "2"
 		)
@@
 			)
 		)
-		(property "LCSC Part #" "C2176190"
+		(property "LCSC Part #" "C161305 "
 			(at 121.92 232.41 90)
 			(effects
@@
 			)
 		)
-		(property "LCSC Part #" "C3832658"
+		(property "LCSC Part #" "C76947 "
 			(at 254 53.34 90)
 			(effects
@@
 			)
 		)
-		(property "LCSC Part #" "C2176190"
+		(property "LCSC Part #" "C161305 "
 			(at 41.91 247.65 90)
 			(effects
@@
 			)
 		)
-		(property "LCSC Part #" "C2661857"
+		(property "LCSC Part #" "C41556732 "
 			(at 316.23 224.79 0)
 			(effects
@@
 			)
 		)
-		(property "LCSC Part #" "C3832658"
+		(property "LCSC Part #" "C76947 "
 			(at 369.57 54.61 0)
 			(effects
@@
 			)
 		)
-		(property "LCSC Part #" "C12530"
+		(property "LCSC Part #" "C77002 "
 			(at 381 232.41 90)
 			(effects
@@
 			)
 		)
-		(property "LCSC Part #" "C12530"
+		(property "LCSC Part #" "C77002 "
 			(at 345.44 231.14 90)
 			(effects
