File: BAgmenzi/tx.kicad_sch (KiCad schematic)
At the start: 29 parts, among them Q1 NX7002BKMBYL, U7 LT3463AEDD#PBF, U8 TPS22916CYFPR

Commit message: added libraries, other changes in sch, started pcb
Parts:
- added JP6: SolderJumper_3_Open, symbol Jumper:SolderJumper_3_Open
- C35: renamed from C34; footprint (none) -> Capacitor_SMD:C_0402_1005Metric
- C36: renamed from C35; value 2.2u -> 2.2u 50V; footprint (none) -> Capacitor_SMD:C_0402_1005Metric
- C37: renamed from C36; footprint (none) -> Capacitor_SMD:C_0402_1005Metric
- C38: renamed from C37; footprint (none) -> Capacitor_SMD:C_0402_1005Metric
- C39: renamed from C38; footprint (none) -> Capacitor_SMD:C_0402_1005Metric
- C41: renamed from C40; footprint (none) -> Capacitor_SMD:C_0402_1005Metric
- C42: renamed from C41; footprint (none) -> Capacitor_SMD:C_0402_1005Metric
- C43: renamed from C42; footprint Capacitor_SMD:C_0201_0603Metric -> Capacitor_SMD:C_0402_1005Metric
- D2: footprint (none) -> Diode_SMD:D_SOD-323_HandSoldering
- FB1, FB2: footprint (none) -> Inductor_SMD:L_0603_1608Metric
- L5, L6: footprint C__Users_Public_Documents_Altium_Projects_PcbLib1.PcbLib:INDC1005X45N -> wulpus:INDC1005X45N
- Q1: footprint (none) -> wulpus_pro_acq:NX7002BKMBYL
- R11oderC_direct1, R17, R18, R19, R24, R25: footprint (none) -> Resistor_SMD:R_0402_1005Metric
- R20, R21, R22, R23: footprint Resistor_SMD:R_0201_0603Metric -> Resistor_SMD:R_0402_1005Metric
- TP7: footprint (none) -> EEG_PcbLib:TEST_POINT_KEYSTONE_5007_TRAD
- renumbered C39 to C40
Connections:
- net V_SYS: now also JP6.3 (B); no longer U8.A2 (VIN)
- new net: JP6.2 (C), U8.A2 (VIN)
- new net V_BAT: JP6.1 (A)
Other:
- moved on the sheet: U8

Commit message: changed VRX rail and deleted U12
Parts:
- added C33: 0.1u 50V, Capacitor_SMD:C_0201_0603Metric, symbol Device:C
- added R14: 100k, Resistor_SMD:R_0402_1005Metric, symbol Device:R
- JP6: footprint (none) -> Jumper:SolderJumper-3_P1.3mm_Open_Pad1.0x1.5mm
Connections:
- net GND: now also R14.2
- net HV_NEG_EN: no longer D2.1 (K), L6.2, R24.1, U7.4 (SW2), U7.5 (D2), U7.9 (~{SHDN1})
- net HV_PWR_EN: now also R14.1
- net PULSE_EN_N renamed PULSER_HIZ_IN
- net PULSE_HV_OUT renamed PULSE_HV
- net PULSE_LV_IN renamed PULSE_OUT
- new net: C33.2, L6.2, U7.4 (SW2)
- new net: C33.1, D2.1 (K), U7.5 (D2)
- new net HV_POS_EN: R24.1, U7.9 (~{SHDN1})
Other:
- moved on the sheet: R24, R25

Commit message: started layout, front v backside
Parts:
- C33: footprint Capacitor_SMD:C_0201_0603Metric -> Capacitor_SMD:C_0402_1005Metric
- TP7: footprint EEG_PcbLib:TEST_POINT_KEYSTONE_5007_TRAD -> TestPoint:TestPoint_THTPad_1.0x1.0mm_Drill0.5mm
Changed lines of the file:
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@@
 	(paper "A4")
 	(rectangle
-		(start 22.86 25.4)
+		(start 19.05 25.4)
 		(end 81.28 78.74)
 		(stroke
@@
 			)
 		)
-		(property "Footprint" "Capacitor_SMD:C_0201_0603Metric"
+		(property "Footprint" "Capacitor_SMD:C_0402_1005Metric"
 			(at 81.28 148.2852 0)
 			(effects
@@
 			)
 		)
-		(property "Footprint" "EEG_PcbLib:TEST_POINT_KEYSTONE_5007_TRAD"
+		(property "Footprint" "TestPoint:TestPoint_THTPad_1.0x1.0mm_Drill0.5mm"
 			(at 36.83 100.33 0)
 			(effects

Commit message: started routing, changed enable signals to nRF
Parts:
- C40: footprint Capacitor_SMD:C_0201_0603Metric -> Capacitor_SMD:C_0402_1005Metric
Changed lines of the file:
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@@
 			)
 		)
-		(property "Footprint" "Capacitor_SMD:C_0201_0603Metric"
+		(property "Footprint" "Capacitor_SMD:C_0402_1005Metric"
 			(at 129.2352 113.03 0)
 			(effects

Commit message: routed msp and nrf
Connections:
- net PULSER_IN: no longer R17.2
- net PULSE_OUT: no longer R17.1
Other:
- moved on the sheet: R17
Changed lines of the file:
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@@
 	(symbol
 		(lib_id "Device:R")
-		(at 52.07 35.56 90)
+		(at 52.07 35.56 180)
 		(unit 1)
 		(exclude_from_sim no)
@@
 		(fields_autoplaced yes)
 		(property "Reference" "R17"
-			(at 52.07 29.21 90)
+			(at 54.61 34.2899 0)
 			(effects
 				(font
 					(size 1.27 1.27)
 				)
+				(justify right)
 			)
 		)
 		(property "Value" "51"
-			(at 52.07 31.75 90)
+			(at 54.61 36.8299 0)
 			(effects
 				(font
 					(size 1.27 1.27)
 				)
+				(justify right)
 			)
 		)
 		(property "Footprint" "Resistor_SMD:R_0402_1005Metric"
-			(at 52.07 37.338 90)
+			(at 53.848 35.56 90)
 			(effects
 				(font

Commit message: DRC correfted all red falgs
Parts:
- removed TP7: +V_hv_in, TestPoint:TestPoint_THTPad_1.0x1.0mm_Drill0.5mm, symbol Connector:TestPoint
Connections:
- net PULSER_IN: now also R17.1
- net PULSE_OUT: now also R17.2
Other:
- moved on the sheet: R17
Changed lines of the file:
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@@
 	(symbol
 		(lib_id "Device:R")
-		(at 52.07 35.56 180)
+		(at 52.07 35.56 270)
 		(unit 1)
 		(exclude_from_sim no)
@@
 		(on_board yes)
 		(dnp no)
-		(fields_autoplaced yes)
 		(property "Reference" "R17"
-			(at 54.61 34.2899 0)
+			(at 50.7999 33.02 0)
 			(effects
 				(font
@@
 		)
 		(property "Value" "51"
-			(at 54.61 36.8299 0)
+			(at 53.3399 33.02 0)
 			(effects
 				(font
@@
 		)
 		(property "Footprint" "Resistor_SMD:R_0402_1005Metric"
-			(at 53.848 35.56 90)
+			(at 52.07 33.782 90)
 			(effects
 				(font
@@
 					(unit 1)
 				)
-			)
-		)
-	)
-	(symbol
-		(lib_id "Connector:TestPoint")
-		(at 36.83 105.41 90)
-		(unit 1)
-		(exclude_from_sim no)
-		(in_bom yes)
-		(on_board yes)
-		(dnp no)
-		(fields_autoplaced yes)
-		(property "Reference" "TP7"
-			(at 33.528 100.33 90)
-			(effects
-				(font
-					(size 1.27 1.27)
-				)
-			)
-		)
-		(property "Value" "+V_hv_in"
-			(at 33.528 102.87 90)
-			(effects
-				(font
-					(size 1.27 1.27)
-				)
-			)
-		)
-		(property "Footprint" "TestPoint:TestPoint_THTPad_1.0x1.0mm_Drill0.5mm"
-			(at 36.83 100.33 0)
-			(effects
-				(font
-					(size 1.27 1.27)
-				)
-				(hide yes)
-			)
-		)
-		(property "Datasheet" "~"
-			(at 36.83 100.33 0)
-			(effects
-				(font
-					(size 1.27 1.27)
-				)
-				(hide yes)
-			)
-		)
-		(property "Description" "test point"
-			(at 36.83 105.41 0)
-			(effects
-				(font
-					(size 1.27 1.27)
-				)
-				(hide yes)
-			)
-		)
-		(pin "1"
-		)
-		(instances
-			(project ""
-				(path "/8cc4acae-3f14-463c-b0a0-3bc1c8d05954/8e6e7503-3da7-4d51-9f66-311eb0e59877"
-					(reference "TP7")
-					(unit 1)
-				)

Commit message: part numbers added
Parts:
- B1: LCSC Part # (none) -> C2653792
- C33: LCSC Part # (none) -> C53084447
- C35, C36, C37, C38, C40, C41, C42, C43: footprint Capacitor_SMD:C_0402_1005Metric -> Capacitor_SMD:C_0603_1608Metric; LCSC Part # (none) -> C126632
- C39: LCSC Part # (none) -> C20441333
- D2: LCSC Part # (none) -> C460116
- L5, L6: LCSC Part # (none) -> C5452416
- Q1: LCSC Part # (none) -> C478246
- R14: LCSC Part # (none) -> C723496
- R17: LCSC Part # (none) -> C778407
- R18: value 1OK -> 10k; LCSC Part # (none) -> C270305
- R19: value 10K -> 10k; LCSC Part # (none) -> C270305
- R20, R23: LCSC Part # (none) -> C473625
- R21: LCSC Part # (none) -> C325948
- R22: LCSC Part # (none) -> C325619
- R24, R25: LCSC Part # (none) -> C270305
- R71: renamed from R11oderC_direct1; value 0Ohm, oder 10nF 100V -> 0; LCSC Part # (none) -> C364372
- U7: LCSC Part # (none) -> C117169
- U8: LCSC Part # (none) -> C2680319

Commit message: LCSC parts complete, changed L5andL6 footprint
Parts:
- B1: LCSC Part # C2653792 -> C2653792
- C33: LCSC Part # C53084447 -> C913614
- C35, C36, C37, C38, C40, C41, C42, C43: LCSC Part # C126632 -> C668357
- C39: LCSC Part # C20441333 -> C14445
- D2: LCSC Part # C460116 -> C460116
- FB1, FB2: LCSC Part # (none) -> C3717002
- L5, L6: footprint wulpus:INDC1005X45N -> wulpus_pro_acq:FP-LQH3NPH_ME-MFG; LCSC Part # C5452416 -> C701168
- R14: LCSC Part # C723496 -> C192169
- R17: LCSC Part # C778407 -> C482204
- R18, R19, R24, R25: LCSC Part # C270305 -> C191984
- R20, R23: LCSC Part # C473625 -> C413126
- R21: LCSC Part # C325948 -> C278596
- R22: LCSC Part # C325619 -> C416536
- R71: LCSC Part # C364372 -> C190119
- U7: LCSC Part # C117169 -> C580060
Changed lines of the file:
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@@
 		)
 	)
+	(text_box "ist nicht der gleiche Treiber, wie bei WULPUS-PRO, funktioniert mit nur einem Kanal. Sonst gleich"
+		(exclude_from_sim no)
+		(at 128.27 58.42 0)
+		(size 31.75 12.7)
+		(margins 0.9525 0.9525 0.9525 0.9525)
+		(stroke
+			(width 0)
+			(type solid)
+		)
+		(fill
+			(type color)
+			(color 111 245 255 1)
+		)
+		(effects
+			(font
+				(size 1.27 1.27)
+			)
+			(justify left top)
+		)
+	)
 	(text_box "for direct filtering (-HV)we need C to shield pulser from -HV. with indirect biasing we dont need it. \n\nD_direct: 10nF"
 		(exclude_from_sim no)
@@
 			)
 		)
-		(property "LCSC Part #" "C270305"
+		(property "LCSC Part #" "C191984 "
 			(at 50.8 63.5 0)
 			(effects
@@
 			)
 		)
-		(property "LCSC Part #" "C270305"
+		(property "LCSC Part #" "C191984 "
 			(at 58.42 146.05 0)
 			(effects
@@
 			)
 		)
-		(property "LCSC Part #" "C325619"
+		(property "LCSC Part #" "C416536 "
 			(at 107.95 124.46 90)
 			(effects
@@
 			)
 		)
-		(property "LCSC Part #" "C270305"
+		(property "LCSC Part #" "C191984 "
 			(at 68.58 41.91 0)
 			(effects
@@
 			)
 		)
-		(property "LCSC Part #" "C364372"
+		(property "LCSC Part #" "C190119 "
 			(at 231.14 45.72 90)
 			(effects
@@
 			)
 		)
-		(property "LCSC Part #" "C325948"
+		(property "LCSC Part #" "C278596 "
 			(at 116.84 114.3 90)
 			(effects
@@
 			)
 		)
-		(property "LCSC Part #" "C126632"
+		(property "LCSC Part #" "C668357 "
 			(at 156.21 38.1 90)
 			(effects
@@
 			)
 		)
-		(property "LCSC Part #" "C20441333"
+		(property "LCSC Part #" "C14445 "
 			(at 36.83 109.22 0)
 			(effects
@@
 			)
 		)
-		(property "LCSC Part #" "C126632"
+		(property "LCSC Part #" "C668357 "
 			(at 203.2 105.41 0)
 			(effects
@@
 			)
 		)
-		(property "LCSC Part #" "C126632"
+		(property "LCSC Part #" "C668357 "
 			(at 196.85 36.83 90)
 			(effects
@@
 			)
 		)
-		(property "LCSC Part #" "C126632"
+		(property "LCSC Part #" "C668357 "
 			(at 231.14 139.7 0)
 			(effects
@@
 			)
 		)
+		(property "LCSC Part #" "C3717002 "
+			(at 215.9 96.52 90)
+			(effects
+				(font
+					(size 1.27 1.27)
+				)
+				(hide yes)
+			)
+		)
 		(pin "1"
 		)
@@
 			)
 		)
-		(property "Footprint" "wulpus:INDC1005X45N"
+		(property "Footprint" "wulpus_pro_acq:FP-LQH3NPH_ME-MFG"
 			(at 50.8 121.92 0)
 			(effects
@@
 			)
 		)
-		(property "LCSC Part #" "C5452416"
+		(property "LCSC Part #" "C701168 "
 			(at 50.8 121.92 0)
 			(effects
@@
 			)
 		)
-		(property "LCSC Part #" "C126632"
+		(property "LCSC Part #" "C668357 "
 			(at 138.43 149.86 0)
 			(effects
@@
 			)
 		)
-		(property "LCSC Part #" "C117169"
+		(property "LCSC Part #" "C580060 "
 			(at 73.66 109.22 0)
 			(effects
@@
 			)
 		)
-		(property "LCSC Part #" "C723496"
+		(property "LCSC Part #" "C192169 "
 			(at 91.44 180.34 0)
 			(effects
@@
 			)
 		)
-		(property "LCSC Part #" "C53084447 "
+		(property "LCSC Part #" "C913614 "
 			(at 85.09 147.32 90)
 			(effects
@@
 			)
 		)
-		(property "LCSC Part #" "C270305"
+		(property "LCSC Part #" "C191984 "
 			(at 49.53 146.05 0)
 			(effects
@@
 			)
 		)
-		(property "LCSC Part #" "C460116"
+		(property "LCSC Part #" "C460116 "
 			(at 118.11 139.7 0)
 			(effects
@@
 			)
 		)
-		(property "LCSC Part #" "C126632"
+		(property "LCSC Part #" "C668357 "
 			(at 128.27 109.22 0)
 			(effects
@@
 			)
 		)
-		(property "LCSC Part #" "C778407"
+		(property "LCSC Part #" "C482204 "
 			(at 52.07 35.56 0)
 			(effects
@@
 			)
 		)
-		(property "LCSC Part #" " C473625"
+		(property "LCSC Part #" "C413126 "
 			(at 127 130.81 0)
 			(effects
@@
 			)
 		)
-		(property "LCSC Part #" " C473625"
+		(property "LCSC Part #" "C413126 "
 			(at 109.22 107.95 0)
 			(effects
@@
 			)
 		)
-		(property "LCSC Part #" "C126632"
+		(property "LCSC Part #" "C668357 "
 			(at 204.47 139.7 0)
 			(effects
@@
 			)
 		)
+		(property "LCSC Part #" "C3717002 "
+			(at 217.17 130.81 90)
+			(effects
+				(font
+					(size 1.27 1.27)
+				)
+				(hide yes)
+			)
+		)
 		(pin "1"
 		)
@@
 			)
 		)
-		(property "LCSC Part #" "C126632"
+		(property "LCSC Part #" "C668357 "
 			(at 229.87 105.41 0)
 			(effects
@@
 			)
 		)
-		(property "Footprint" "wulpus:INDC1005X45N"
+		(property "Footprint" "wulpus_pro_acq:FP-LQH3NPH_ME-MFG"
 			(at 50.8 130.81 0)
 			(effects
@@
 			)
 		)
-		(property "LCSC Part #" "C5452416"
+		(property "LCSC Part #" "C701168 "
 			(at 50.8 130.81 0)
 			(effects
@@
 			)
 		)
-		(property "LCSC Part #" "C2653792"
+		(property "LCSC Part #" "C2653792 "
 			(at 160.02 41.91 0)
 			(effects
