File: BAgmenzi/tx.kicad_sch (KiCad schematic)
At the start: 31 parts, among them Q1 NX7002BKMBYL, U7 LT3463AEDD#PBF, U8 TPS22916CYFPR

Commit message: corrected LCSC numbers, other changes, Testpoints
Parts:
- added +HV2, -HV1: TestPoint, TestPoint:TestPoint_Pad_D1.0mm, symbol Connector:TestPoint
- B1: LCSC Part # C2653792 -> C2653792
- C33: LCSC Part # C913614 -> C913614
- C35, C36, C37, C38, C40, C41, C42, C43: LCSC Part # C668357 -> C668357
- C39: LCSC Part # C14445 -> C14445
- D2: LCSC Part # C460116 -> C460116
- FB1, FB2: LCSC Part # C3717002 -> C3717002
- L5, L6: value LQG15HS3N9B02D -> LQH3NPZ100MMEL; LCSC Part # C701168 -> C701168
- R14: LCSC Part # C192169 -> C192169
- R17: LCSC Part # C482204 -> C482204
- R18, R19, R24, R25: LCSC Part # C191984 -> C191984
- R20, R23: LCSC Part # C413126 -> C413126
- R21: LCSC Part # C278596 -> C278596
- R22: LCSC Part # C416536 -> C416536
- R71: LCSC Part # C190119 -> C190119
- U7: LCSC Part # C580060 -> C580060
Connections:
- net +HV: now also -HV1.1
- net -HV: now also +HV2.1
Changed lines of the file:
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@@
 	)
 	(junction
+		(at 240.03 96.52)
+		(diameter 0)
+		(color 0 0 0 0)
+	)
+	(junction
 		(at 109.22 139.7)
 		(diameter 0)
@@
 	(wire
 		(pts
-			(xy 190.5 36.83) (xy 190.5 30.48)
+			(xy 190.5 36.83) (xy 190.5 29.21)
 		)
 		(stroke
@@
 	(wire
 		(pts
-			(xy 229.87 96.52) (xy 254 96.52)
+			(xy 229.87 96.52) (xy 240.03 96.52)
 		)
 		(stroke
@@
 	(wire
 		(pts
+			(xy 240.03 96.52) (xy 254 96.52)
+		)
+		(stroke
+			(width 0)
+			(type default)
+		)
+	)
+	(wire
+		(pts
 			(xy 132.08 100.33) (xy 132.08 104.14)
 		)
@@
 			)
 		)
-		(property "LCSC Part #" "C191984 "
+		(property "LCSC Part #" "C191984"
 			(at 50.8 63.5 0)
 			(effects
@@
 			)
 		)
-		(property "LCSC Part #" "C191984 "
+		(property "LCSC Part #" "C191984"
 			(at 58.42 146.05 0)
 			(effects
@@
 			)
 		)
-		(property "LCSC Part #" "C416536 "
+		(property "LCSC Part #" "C416536"
 			(at 107.95 124.46 90)
 			(effects
@@
 			)
 		)
-		(property "LCSC Part #" "C191984 "
+		(property "LCSC Part #" "C191984"
 			(at 68.58 41.91 0)
 			(effects
@@
 			)
 		)
-		(property "LCSC Part #" "C190119 "
+		(property "LCSC Part #" "C190119"
 			(at 231.14 45.72 90)
 			(effects
@@
 			)
 		)
-		(property "LCSC Part #" "C278596 "
+		(property "LCSC Part #" "C278596"
 			(at 116.84 114.3 90)
 			(effects
@@
 			)
 		)
-		(property "LCSC Part #" "C668357 "
+		(property "LCSC Part #" "C668357"
 			(at 156.21 38.1 90)
 			(effects
@@
 			)
 		)
-		(property "LCSC Part #" "C14445 "
+		(property "LCSC Part #" "C14445"
 			(at 36.83 109.22 0)
 			(effects
@@
 			)
 		)
-		(property "LCSC Part #" "C668357 "
+		(property "LCSC Part #" "C668357"
 			(at 203.2 105.41 0)
 			(effects
@@
 			)
 		)
-		(property "LCSC Part #" "C668357 "
+		(property "LCSC Part #" "C668357"
 			(at 196.85 36.83 90)
 			(effects
@@
 			)
 		)
-		(property "LCSC Part #" "C668357 "
+		(property "LCSC Part #" "C668357"
 			(at 231.14 139.7 0)
 			(effects
@@
 			)
 		)
-		(property "LCSC Part #" "C3717002 "
+		(property "LCSC Part #" "C3717002"
 			(at 215.9 96.52 90)
 			(effects
@@
 			)
 		)
-		(property "Value" "LQG15HS3N9B02D"
+		(property "Value" "LQH3NPZ100MMEL"
 			(at 51.562 117.602 0)
 			(effects
@@
 			)
 		)
-		(property "LCSC Part #" "C701168 "
+		(property "LCSC Part #" "C701168"
 			(at 50.8 121.92 0)
 			(effects
@@
 	)
 	(symbol
+		(lib_id "Connector:TestPoint")
+		(at 240.03 96.52 0)
+		(unit 1)
+		(exclude_from_sim no)
+		(in_bom yes)
+		(on_board yes)
+		(dnp no)
+		(fields_autoplaced yes)
+		(property "Reference" "+HV2"
+			(at 242.57 91.9479 0)
+			(effects
+				(font
+					(size 1.27 1.27)
+				)
+				(justify left)
+			)
+		)
+		(property "Value" "TestPoint"
+			(at 242.57 94.4879 0)
+			(effects
+				(font
+					(size 1.27 1.27)
+				)
+				(justify left)
+			)
+		)
+		(property "Footprint" "TestPoint:TestPoint_Pad_D1.0mm"
+			(at 245.11 96.52 0)
+			(effects
+				(font
+					(size 1.27 1.27)
+				)
+				(hide yes)
+			)
+		)
+		(property "Datasheet" "~"
+			(at 245.11 96.52 0)
+			(effects
+				(font
+					(size 1.27 1.27)
+				)
+				(hide yes)
+			)
+		)
+		(property "Description" "test point"
+			(at 240.03 96.52 0)
+			(effects
+				(font
+					(size 1.27 1.27)
+				)
+				(hide yes)
+			)
+		)
+		(pin "1"
+		)
+		(instances
+			(project "BAgmenzi"
+				(path "/8cc4acae-3f14-463c-b0a0-3bc1c8d05954/8e6e7503-3da7-4d51-9f66-311eb0e59877"
+					(reference "+HV2")
+					(unit 1)
+				)
+			)
+		)
+	)
+	(symbol
 		(lib_id "Device:C")
 		(at 138.43 149.86 0)
@@
 			)
 		)
-		(property "LCSC Part #" "C668357 "
+		(property "LCSC Part #" "C668357"
 			(at 138.43 149.86 0)
 			(effects
@@
 			)
 		)
-		(property "LCSC Part #" "C580060 "
+		(property "LCSC Part #" "C580060"
 			(at 73.66 109.22 0)
 			(effects
@@
 			)
 		)
-		(property "LCSC Part #" "C192169 "
+		(property "LCSC Part #" "C192169"
 			(at 91.44 180.34 0)
 			(effects
@@
 			)
 		)
-		(property "LCSC Part #" "C913614 "
+		(property "LCSC Part #" "C913614"
 			(at 85.09 147.32 90)
 			(effects
@@
 	)
 	(symbol
+		(lib_id "Connector:TestPoint")
+		(at 160.02 26.67 0)
+		(unit 1)
+		(exclude_from_sim no)
+		(in_bom yes)
+		(on_board yes)
+		(dnp no)
+		(fields_autoplaced yes)
+		(property "Reference" "-HV1"
+			(at 162.56 22.0979 0)
+			(effects
+				(font
+					(size 1.27 1.27)
+				)
+				(justify left)
+			)
+		)
+		(property "Value" "TestPoint"
+			(at 162.56 24.6379 0)
+			(effects
+				(font
+					(size 1.27 1.27)
+				)
+				(justify left)
+			)
+		)
+		(property "Footprint" "TestPoint:TestPoint_Pad_D1.0mm"
+			(at 165.1 26.67 0)
+			(effects
+				(font
+					(size 1.27 1.27)
+				)
+				(hide yes)
+			)
+		)
+		(property "Datasheet" "~"
+			(at 165.1 26.67 0)
+			(effects
+				(font
+					(size 1.27 1.27)
+				)
+				(hide yes)
+			)
+		)
+		(property "Description" "test point"
+			(at 160.02 26.67 0)
+			(effects
+				(font
+					(size 1.27 1.27)
+				)
+				(hide yes)
+			)
+		)
+		(pin "1"
+		)
+		(instances
+			(project "BAgmenzi"
+				(path "/8cc4acae-3f14-463c-b0a0-3bc1c8d05954/8e6e7503-3da7-4d51-9f66-311eb0e59877"
+					(reference "-HV1")
+					(unit 1)
+				)
+			)
+		)
+	)
+	(symbol
 		(lib_id "power:GND")
 		(at 101.6 179.07 0)
@@
 			)
 		)
-		(property "LCSC Part #" "C191984 "
+		(property "LCSC Part #" "C191984"
 			(at 49.53 146.05 0)
 			(effects
@@
 			)
 		)
-		(property "LCSC Part #" "C460116 "
+		(property "LCSC Part #" "C460116"
 			(at 118.11 139.7 0)
 			(effects
@@
 			)
 		)
-		(property "LCSC Part #" "C668357 "
+		(property "LCSC Part #" "C668357"
 			(at 128.27 109.22 0)
 			(effects
@@
 			)
 		)
-		(property "LCSC Part #" "C482204 "
+		(property "LCSC Part #" "C482204"
 			(at 52.07 35.56 0)
 			(effects
@@
 			)
 		)
-		(property "LCSC Part #" "C413126 "
+		(property "LCSC Part #" "C413126"
 			(at 127 130.81 0)
 			(effects
@@
 			)
 		)
-		(property "LCSC Part #" "C413126 "
+		(property "LCSC Part #" "C413126"
 			(at 109.22 107.95 0)
 			(effects
@@
 			)
 		)
-		(property "LCSC Part #" "C668357 "
+		(property "LCSC Part #" "C668357"
 			(at 204.47 139.7 0)
 			(effects
@@
 			)
 		)
-		(property "LCSC Part #" "C3717002 "
+		(property "LCSC Part #" "C3717002"
 			(at 217.17 130.81 90)
 			(effects
@@
 			)
 		)
-		(property "LCSC Part #" "C668357 "
+		(property "LCSC Part #" "C668357"
 			(at 229.87 105.41 0)
 			(effects
@@
 			)
 		)
-		(property "Value" "LQG15HS3N9B02D"
+		(property "Value" "LQH3NPZ100MMEL"
 			(at 51.562 126.492 0)
 			(effects
@@
 			)
 		)
-		(property "LCSC Part #" "C701168 "
+		(property "LCSC Part #" "C701168"
 			(at 50.8 130.81 0)
 			(effects
@@
 			)
 		)
-		(property "LCSC Part #" "C2653792 "
+		(property "LCSC Part #" "C2653792"
 			(at 160.02 41.91 0)
 			(effects

Commit message: small changes
Parts:
- +HV1: renamed from -HV1; now left out of the parts list
- -HV2: renamed from +HV2; now left out of the parts list
Changed lines of the file:
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@@
 		(unit 1)
 		(exclude_from_sim no)
-		(in_bom yes)
+		(in_bom no)
 		(on_board yes)
 		(dnp no)
 		(fields_autoplaced yes)
-		(property "Reference" "+HV2"
+		(property "Reference" "-HV2"
 			(at 242.57 91.9479 0)
 			(effects
@@
 			(project "BAgmenzi"
 				(path "/8cc4acae-3f14-463c-b0a0-3bc1c8d05954/8e6e7503-3da7-4d51-9f66-311eb0e59877"
-					(reference "+HV2")
+					(reference "-HV2")
 					(unit 1)
 				)
@@
 		(unit 1)
 		(exclude_from_sim no)
-		(in_bom yes)
+		(in_bom no)
 		(on_board yes)
 		(dnp no)
 		(fields_autoplaced yes)
-		(property "Reference" "-HV1"
+		(property "Reference" "+HV1"
 			(at 162.56 22.0979 0)
 			(effects
@@
 			(project "BAgmenzi"
 				(path "/8cc4acae-3f14-463c-b0a0-3bc1c8d05954/8e6e7503-3da7-4d51-9f66-311eb0e59877"
-					(reference "-HV1")
+					(reference "+HV1")
 					(unit 1)
 				)
