File: BAgmenzi/cmut.kicad_sch (KiCad schematic)
At the start: 14 parts, among them U5 polyCMUT

Commit message: small changes
Parts:
- U5: now not fitted
Connections:
- net GND: no longer U5.1 (GND)
- net PULSE_HV: now also U5.4 (CH3); no longer U5.5 (CH4)
- net RX_IN: now also U5.7 (CH6); no longer U5.8 (CH7)
- net at JP5.2 (C), TP8.1: now also U5.1 (GND); no longer U5.2 (CH1)
Changed lines of the file:
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@@
 		)
 	)
-	(text_box "the common electrode is on pad 1\nTX is on pad 4\nRX is on pad 7"
+	(text_box "the common electrode is on pad 1\nTX is on pad 4\nRX is on pad 7\n\nBOT_EL = GND (?)"
 		(exclude_from_sim no)
 		(at 193.04 113.03 0)
@@
 	)
 	(no_connect
-		(at 191.77 86.36)
+		(at 191.77 81.28)
 	)
 	(no_connect
-		(at 191.77 81.28)
+		(at 191.77 91.44)
 	)
 	(no_connect
@@
 	)
 	(no_connect
-		(at 191.77 93.98)
+		(at 191.77 83.82)
 	)
 	(no_connect
@@
 	(wire
 		(pts
+			(xy 173.99 86.36) (xy 173.99 85.09)
+		)
+		(stroke
+			(width 0)
+			(type default)
+		)
+	)
+	(wire
+		(pts
 			(xy 130.81 135.89) (xy 134.62 135.89)
 		)
@@
 	(wire
 		(pts
-			(xy 173.99 85.09) (xy 173.99 83.82)
-		)
-		(stroke
-			(width 0)
-			(type default)
-		)
-	)
-	(wire
-		(pts
 			(xy 127 119.38) (xy 130.81 119.38)
 		)
@@
 	(wire
 		(pts
+			(xy 180.34 93.98) (xy 180.34 91.44)
+		)
+		(stroke
+			(width 0)
+			(type default)
+		)
+	)
+	(wire
+		(pts
 			(xy 134.62 135.89) (xy 138.43 135.89)
 		)
@@
 	(wire
 		(pts
-			(xy 88.9 91.44) (xy 191.77 91.44)
+			(xy 88.9 91.44) (xy 180.34 91.44)
 		)
 		(stroke
@@
 	(wire
 		(pts
+			(xy 191.77 86.36) (xy 173.99 86.36)
+		)
+		(stroke
+			(width 0)
+			(type default)
+		)
+	)
+	(wire
+		(pts
 			(xy 134.62 85.09) (xy 173.99 85.09)
 		)
@@
 	(wire
 		(pts
+			(xy 191.77 93.98) (xy 180.34 93.98)
+		)
+		(stroke
+			(width 0)
+			(type default)
+		)
+	)
+	(wire
+		(pts
 			(xy 68.58 87.63) (xy 88.9 87.63)
 		)
@@
 	(wire
 		(pts
-			(xy 173.99 83.82) (xy 191.77 83.82)
-		)
-		(stroke
-			(width 0)
-			(type default)
-		)
-	)
-	(wire
-		(pts
 			(xy 132.08 46.99) (xy 132.08 53.34)
 		)
@@
 	(wire
 		(pts
-			(xy 144.78 99.06) (xy 191.77 99.06)
+			(xy 144.78 100.33) (xy 191.77 100.33)
 		)
 		(stroke
@@
 	(wire
 		(pts
-			(xy 144.78 99.06) (xy 144.78 104.14)
-		)
-		(stroke
-			(width 0)
-			(type default)
-		)
-	)
-	(wire
-		(pts
-			(xy 186.69 101.6) (xy 191.77 101.6)
+			(xy 144.78 100.33) (xy 144.78 104.14)
+		)
+		(stroke
+			(width 0)
+			(type default)
+		)
+	)
+	(wire
+		(pts
+			(xy 191.77 100.33) (xy 191.77 101.6)
 		)
 		(stroke
@@
 		(in_bom yes)
 		(on_board yes)
-		(dnp no)
+		(dnp yes)
 		(fields_autoplaced yes)
 		(property "Reference" "U5"
@@
 					(unit 1)
 				)
-			)
-		)
-	)
-	(symbol
-		(lib_id "power:GND")
-		(at 186.69 101.6 0)
-		(unit 1)
-		(exclude_from_sim no)
-		(in_bom yes)
-		(on_board yes)
-		(dnp no)
-		(fields_autoplaced yes)
-		(property "Reference" "#PWR091"
-			(at 186.69 107.95 0)
-			(effects
-				(font
-					(size 1.27 1.27)
-				)
-				(hide yes)
-			)
-		)
-		(property "Value" "GND"
-			(at 186.69 106.68 0)
-			(effects
-				(font
-					(size 1.27 1.27)
-				)
-			)
-		)
-		(property "Footprint" ""
-			(at 186.69 101.6 0)
-			(effects
-				(font
-					(size 1.27 1.27)
-				)
-				(hide yes)
-			)
-		)
-		(property "Datasheet" ""
-			(at 186.69 101.6 0)
-			(effects
-				(font
-					(size 1.27 1.27)
-				)
-				(hide yes)
-			)
-		)
-		(property "Description" "Power symbol creates a global label with name \"GND\" , ground"
-			(at 186.69 101.6 0)
-			(effects
-				(font
-					(size 1.27 1.27)
-				)
-				(hide yes)
-			)
-		)
-		(pin "1"
-		)
-		(instances
-			(project ""
-				(path "/8cc4acae-3f14-463c-b0a0-3bc1c8d05954/edb8e8bc-fb53-4a31-8600-d64a48325b03"
-					(reference "#PWR091")
-					(unit 1)
-				)
