File: BAgmenzi/nrf.kicad_sch (KiCad schematic)
At the start: 10 parts, among them J5 3220-10-0100-00

Commit message: part numbers added
Parts:
- C55, C66: LCSC Part # (none) -> C161362
- C64, C65: LCSC Part # (none) -> C23733
- J5: LCSC Part # (none) -> C5154224
- R45, R46: LCSC Part # (none) -> C25091
- R47, R48: LCSC Part # (none) -> C606165
Connections:
- net PPG_I2C.SDA: now also M1.G3 (P128); no longer M1.G8 (P108)
Changed lines of the file:
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@@
 	)
 	(no_connect
+		(at 257.81 121.92)
+	)
+	(no_connect
 		(at 161.29 40.64)
 	)
@@
 	)
 	(no_connect
-		(at 257.81 109.22)
-	)
-	(no_connect
 		(at 257.81 40.64)
 	)
@@
 	(wire
 		(pts
-			(xy 267.97 106.68) (xy 257.81 106.68)
+			(xy 274.32 106.68) (xy 257.81 106.68)
 		)
 		(stroke
@@
 	(wire
 		(pts
-			(xy 274.32 121.92) (xy 257.81 121.92)
+			(xy 274.32 109.22) (xy 257.81 109.22)
 		)
 		(stroke
@@
 	)
 	(label "nRST"
-		(at 267.97 106.68 180)
+		(at 274.32 106.68 180)
 		(effects
 			(font
@@
 		)
 	)
-	(label "PPG_I2C.SDA"
-		(at 274.32 121.92 180)
-		(effects
-			(font
-				(size 1.27 1.27)
-			)
-			(justify right bottom)
-		)
-	)
 	(label "SWCLK"
 		(at 269.24 33.02 180)
@@
 		)
 	)
+	(label "PPG_I2C.SDA"
+		(at 274.32 109.22 180)
+		(effects
+			(font
+				(size 1.27 1.27)
+			)
+			(justify right bottom)
+		)
+	)
 	(label "nRST"
 		(at 88.9 173.99 180)
@@
 			)
 		)
+		(property "LCSC Part #" "C25091"
+			(at 72.39 167.64 90)
+			(effects
+				(font
+					(size 1.27 1.27)
+				)
+				(hide yes)
+			)
+		)
 		(pin "2"
 		)
@@
 			)
 		)
+		(property "LCSC Part #" "C161362"
+			(at 140.97 96.52 0)
+			(effects
+				(font
+					(size 1.27 1.27)
+				)
+				(hide yes)
+			)
+		)
 		(pin "2"
 		)
@@
 			)
 		)
+		(property "LCSC Part #" "C23733"
+			(at 281.94 100.33 0)
+			(effects
+				(font
+					(size 1.27 1.27)
+				)
+				(hide yes)
+			)
+		)
 		(pin "2"
 		)
@@
 			)
 		)
+		(property "LCSC Part #" "C606165"
+			(at 214.63 153.67 0)
+			(effects
+				(font
+					(size 1.27 1.27)
+				)
+				(hide yes)
+			)
+		)
 		(pin "1"
 		)
@@
 			)
 		)
+		(property "LCSC Part #" "C23733"
+			(at 151.13 77.47 0)
+			(effects
+				(font
+					(size 1.27 1.27)
+				)
+				(hide yes)
+			)
+		)
 		(pin "2"
 		)
@@
 			)
 		)
+		(property "LCSC Part #" "C161362"
+			(at 149.86 100.33 0)
+			(effects
+				(font
+					(size 1.27 1.27)
+				)
+				(hide yes)
+			)
+		)
 		(pin "2"
 		)
@@
 			)
 		)
+		(property "LCSC Part #" "C606165"
+			(at 217.17 153.67 0)
+			(effects
+				(font
+					(size 1.27 1.27)
+				)
+				(hide yes)
+			)
+		)
 		(pin "1"
 		)
@@
 			)
 		)
+		(property "LCSC Part #" "C25091"
+			(at 72.39 163.83 90)
+			(effects
+				(font
+					(size 1.27 1.27)
+				)
+				(hide yes)
+			)
+		)
 		(pin "2"
 		)
@@
 				)
 				(hide yes)
+			)
+		)
+		(property "LCSC Part #" "C5154224"
+			(at 53.34 168.91 0)
+			(effects
+				(font
+					(size 1.27 1.27)
+				)
+				(hide yes)

Commit message: LCSC parts complete, changed L5andL6 footprint
Parts:
- C55, C66: LCSC Part # C161362 -> C169842
- J5: LCSC Part # C5154224 -> C5154224
- R47, R48: LCSC Part # C606165 -> C11702
Changed lines of the file:
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@@
 			)
 		)
-		(property "LCSC Part #" "C161362"
+		(property "LCSC Part #" "C169842 "
 			(at 140.97 96.52 0)
 			(effects
@@
 			)
 		)
-		(property "LCSC Part #" "C606165"
+		(property "LCSC Part #" "C11702 "
 			(at 214.63 153.67 0)
 			(effects
@@
 			)
 		)
-		(property "LCSC Part #" "C161362"
+		(property "LCSC Part #" "C169842 "
 			(at 149.86 100.33 0)
 			(effects
@@
 			)
 		)
-		(property "LCSC Part #" "C606165"
+		(property "LCSC Part #" "C11702 "
 			(at 217.17 153.67 0)
 			(effects
@@
 			)
 		)
-		(property "LCSC Part #" "C5154224"
+		(property "LCSC Part #" "C5154224 "
 			(at 53.34 168.91 0)
 			(effects

Commit message: corrected LCSC numbers, other changes, Testpoints
Parts:
- C55, C66: LCSC Part # C169842 -> C1525
- J5: LCSC Part # C5154224 -> C5382952
- R47, R48: LCSC Part # C11702 -> C11702
Changed lines of the file:
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@@
 			)
 		)
-		(property "LCSC Part #" "C169842 "
+		(property "LCSC Part #" "C1525"
 			(at 140.97 96.52 0)
 			(effects
@@
 			)
 		)
-		(property "LCSC Part #" "C11702 "
+		(property "LCSC Part #" "C11702"
 			(at 214.63 153.67 0)
 			(effects
@@
 			)
 		)
-		(property "LCSC Part #" "C169842 "
+		(property "LCSC Part #" "C1525"
 			(at 149.86 100.33 0)
 			(effects
@@
 			)
 		)
-		(property "LCSC Part #" "C11702 "
+		(property "LCSC Part #" "C11702"
 			(at 217.17 153.67 0)
 			(effects
@@
 			)
 		)
-		(property "LCSC Part #" "C5154224 "
+		(property "LCSC Part #" "C5382952"
 			(at 53.34 168.91 0)
 			(effects

Commit message: small changes
Parts:
- added TP1: DBG_TX, TestPoint:TestPoint_Pad_D1.0mm, symbol Connector:TestPoint
- M1: value ~ -> DNP; now not fitted
Connections:
- net DBG_TX: now reaches M1.E9 (P116-TXD)
- net DBG_TX: now also TP1.1
- no-connect marks 52 -> 51
Changed lines of the file:
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@@
 	)
 	(no_connect
-		(at 207.01 147.32)
-	)
-	(no_connect
 		(at 219.71 147.32)
 	)
@@
 	(wire
 		(pts
+			(xy 207.01 147.32) (xy 207.01 154.94)
+		)
+		(stroke
+			(width 0)
+			(type default)
+		)
+	)
+	(wire
+		(pts
 			(xy 257.81 93.98) (xy 273.05 93.98)
 		)
@@
 	(wire
 		(pts
+			(xy 198.12 154.94) (xy 207.01 154.94)
+		)
+		(stroke
+			(width 0)
+			(type default)
+		)
+	)
+	(wire
+		(pts
 			(xy 214.63 147.32) (xy 214.63 149.86)
 		)
@@
 		)
 	)
+	(label "DBG_TX"
+		(at 198.12 154.94 0)
+		(effects
+			(font
+				(size 1.27 1.27)
+			)
+			(justify left bottom)
+		)
+	)
 	(label "NRF_SPI.MOSI"
 		(at 107.95 85.09 0)
@@
 	)
 	(symbol
+		(lib_id "Connector:TestPoint")
+		(at 198.12 154.94 0)
+		(unit 1)
+		(exclude_from_sim no)
+		(in_bom no)
+		(on_board yes)
+		(dnp no)
+		(property "Reference" "TP1"
+			(at 198.628 150.114 0)
+			(effects
+				(font
+					(size 1.27 1.27)
+				)
+				(justify left)
+			)
+		)
+		(property "Value" "DBG_TX"
+			(at 198.628 151.892 0)
+			(effects
+				(font
+					(size 1.27 1.27)
+				)
+				(justify left)
+			)
+		)
+		(property "Footprint" "TestPoint:TestPoint_Pad_D1.0mm"
+			(at 203.2 154.94 0)
+			(effects
+				(font
+					(size 1.27 1.27)
+				)
+				(hide yes)
+			)
+		)
+		(property "Datasheet" "~"
+			(at 203.2 154.94 0)
+			(effects
+				(font
+					(size 1.27 1.27)
+				)
+				(hide yes)
+			)
+		)
+		(property "Description" "test point"
+			(at 198.12 154.94 0)
+			(effects
+				(font
+					(size 1.27 1.27)
+				)
+				(hide yes)
+			)
+		)
+		(pin "1"
+		)
+		(instances
+			(project ""
+				(path "/8cc4acae-3f14-463c-b0a0-3bc1c8d05954/a8ba6e7f-774b-4308-a555-46c064980fee"
+					(reference "TP1")
+					(unit 1)
+				)
+			)
+		)
+	)
+	(symbol
 		(lib_id "nRF_LIB-altium-import:root_0_NRF51822-44P_130_*")
 		(at 168.91 15.24 0)
@@
 		(in_bom yes)
 		(on_board yes)
-		(dnp no)
+		(dnp yes)
 		(fields_autoplaced yes)
 		(property "Reference" "M1"
@@
 			)
 		)
-		(property "Value" "~"
+		(property "Value" "DNP"
 			(at 209.55 12.7 0)
 			(effects
